File: Schematic/JudgeRemote/_autosave-JudgeRemote.kicad_sch (KiCad schematic)
At the start: 34 parts, among them J1 Battery IN, J10 Solenoid, J6 I2C Out, SW2 Button A, SW2 Button B, SW2 Button C, SW2 Button D, SW2 Button E, SW2 Button F, SW2 Button G, SW2 Button H, U1 ESP32-DevKitC, U2 Mini360

Commit message: work on schematic and start on light handler code
Connections:
- net Battery Reader: now also U1.5 (VDET_1/GPIO34/ADC1_CH6); no longer U1.3 (SENSOR_VP/GPIO36/ADC1_CH0)
- net Button C: now also U1.12 (MTMS/GPIO14/ADC2_CH6); no longer U1.9 (DAC_1/ADC2_CH8/GPIO25)
- net Button D: now also U1.11 (ADC2_CH7/GPIO27); no longer U1.12 (MTMS/GPIO14/ADC2_CH6)
- net Led A: now also U1.9 (DAC_1/ADC2_CH8/GPIO25); no longer U1.11 (ADC2_CH7/GPIO27)
- no-connect marks 13 -> 15
Changed lines of the file:
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@@
   )
   (no_connect (at 139.7 67.31))
+  (no_connect (at 139.7 46.99))
   (no_connect (at 209.55 49.53))
   (no_connect (at 139.7 74.93))
@@
   (no_connect (at 209.55 44.45))
   (no_connect (at 209.55 41.91))
+  (no_connect (at 139.7 39.37))
   (no_connect (at 209.55 80.01))
   (no_connect (at 139.7 36.83))
@@
     (stroke (width 0) (type default))
   )
+  (wire (pts (xy 128.27 64.77) (xy 139.7 64.77))
+    (stroke (width 0) (type default))
+  )
   (wire (pts (xy 27.94 82.55) (xy 27.94 87.63))
     (stroke (width 0) (type default))
@@
     (stroke (width 0) (type default))
   )
+  (wire (pts (xy 128.27 54.61) (xy 139.7 54.61))
+    (stroke (width 0) (type default))
+  )
   (wire (pts (xy 30.48 30.48) (xy 35.56 30.48))
     (stroke (width 0) (type default))
   )
   (wire (pts (xy 73.66 87.63) (xy 73.66 92.71))
+    (stroke (width 0) (type default))
+  )
+  (wire (pts (xy 128.27 57.15) (xy 139.7 57.15))
+    (stroke (width 0) (type default))
+  )
+  (wire (pts (xy 128.27 69.85) (xy 139.7 69.85))
     (stroke (width 0) (type default))
   )
@@
     (effects (font (size 1.27 1.27)) (justify left bottom))
   )
-  (label "Button D" (at 139.7 62.23 180) (fields_autoplaced)
+  (label "Button D" (at 139.7 59.69 180) (fields_autoplaced)
     (effects (font (size 1.27 1.27)) (justify right bottom))
   )
@@
     (effects (font (size 1.27 1.27)) (justify left bottom))
   )
-  (label "Led B" (at 139.7 57.15 180) (fields_autoplaced)
+  (label "Led B" (at 128.27 57.15 180) (fields_autoplaced)
     (effects (font (size 1.27 1.27)) (justify right bottom))
   )
@@
     (effects (font (size 1.27 1.27)) (justify right bottom))
   )
-  (label "Battery Reader" (at 139.7 39.37 180) (fields_autoplaced)
+  (label "Battery Reader" (at 139.7 44.45 180) (fields_autoplaced)
     (effects (font (size 1.27 1.27)) (justify right bottom))
   )
@@
     (effects (font (size 1.27 1.27)) (justify right bottom))
   )
-  (label "Led D" (at 139.7 64.77 180) (fields_autoplaced)
+  (label "Led D" (at 128.27 64.77 180) (fields_autoplaced)
     (effects (font (size 1.27 1.27)) (justify right bottom))
   )
@@
     (effects (font (size 1.27 1.27)) (justify right bottom))
   )
-  (label "Led C" (at 139.7 69.85 180) (fields_autoplaced)
+  (label "Led C" (at 128.27 69.85 180) (fields_autoplaced)
     (effects (font (size 1.27 1.27)) (justify right bottom))
   )
@@
     (effects (font (size 1.27 1.27)) (justify left bottom))
   )
-  (label "Led A" (at 139.7 59.69 180) (fields_autoplaced)
+  (label "Led A" (at 128.27 54.61 180) (fields_autoplaced)
     (effects (font (size 1.27 1.27)) (justify right bottom))
   )
@@
     (effects (font (size 1.27 1.27)) (justify right bottom))
   )
-  (label "Button C" (at 139.7 54.61 180) (fields_autoplaced)
-    (effects (font (size 1.27 1.27)) (justify right bottom))
-  )
+  (label "Button C" (at 139.7 62.23 180) (fields_autoplaced)
+    (effects (font (size 1.27 1.27)) (justify right bottom))
+  )
